Commit message: define params file launch arguments for custom parameter file
Signed-off-by: quic-chenghen <quic_chenghen@quicinc.com>

File: qrb_ros_robot_base_urdf/urdf/robot_base.urdf (robot description, URDF)
Before this commit: robot robot_base, 3 links, 2 joints
Joints:
- joint laser_joint: origin xyz=${box_length/2-1-laser_radius-0.01} 0 ${0.186-chassis_height} rpy=0 0 ${pi} -> xyz=${box_length/2-laser_radius-0.01} 0 ${0.186-chassis_height-(box_height/2)} rpy=0 0 ${pi}
